File: kicad/3340-VCO.kicad_sch (KiCad schematic)
At the start: 78 parts, among them J3 EuroPower_JST_3P, J4 EURO_PWR_16P, SW1 SW_SPDT, U1 78M05, U1 AS3340, U2 79M05, U2 TL074

Commit message: added schem 0.1.1
Parts:
- added J10: SINE, DIYSynthMNL:AudioJack_3.5mm_long_pads, symbol DIYSynthMNL:PJ3001F
- added J11: PULSE, DIYSynthMNL:AudioJack_3.5mm_long_pads, symbol DIYSynthMNL:PJ3001F
- added J3: FM, DIYSynthMNL:AudioJack_3.5mm_long_pads, symbol DIYSynthMNL:PJ3001F
- added J4: PWM, DIYSynthMNL:AudioJack_3.5mm_long_pads, symbol DIYSynthMNL:PJ3001F
- added J5: Sync, DIYSynthMNL:AudioJack_3.5mm_long_pads, symbol DIYSynthMNL:PJ3001F
- added J6: vOct1, DIYSynthMNL:AudioJack_3.5mm_long_pads, symbol DIYSynthMNL:PJ3001F
- added J7: vOct2, DIYSynthMNL:AudioJack_3.5mm_long_pads, symbol DIYSynthMNL:PJ3001F
- added J8: SAW, DIYSynthMNL:AudioJack_3.5mm_long_pads, symbol DIYSynthMNL:PJ3001F
- added J9: TRI, DIYSynthMNL:AudioJack_3.5mm_long_pads, symbol DIYSynthMNL:PJ3001F
- added RV7: 100K, symbol Device:R_Potentiometer
Connections:
- net GND: now also J10.S, J11.S, J3.S, J4.S, J5.S, J6.S, J7.S, J8.S, J9.S, RV7.1
- net Lin_FM_In: now also RV7.2
- net PWM_In: now also J4.T
- net PWM_normalled: now also J4.TN
- net Pulse_out: now also J11.T
- net Saw_out: now also J8.T
- net Sine_out: now also J10.T
- net Sync_In: now also J5.T
- net Tri_out: now also J9.T
- net V/OCT_In_1: now also J7.T
- net V/OCT_In_2: now also J6.T
- new net: J3.T, RV7.3
- no-connect marks 6 -> 14
Other:
- moved on the sheet: C14, C15, C17, R6, R7, R8, SW1

Commit message: added multiboard schematic (rev 0.1.2)
Parts:
- removed C13: 1nF_Polystyrene, symbol Device:C
- removed C14, C16: 10nF, symbol Device:C
- removed C15, C2, C3: 100nF, symbol Device:C
- removed C17: 1nF, symbol Device:C
- removed C17, C5, C8: 100nF, DIYSynthMNL:C_Rect_L7.0mm_W2.0mm_P5.00mm_BigPads, symbol Device:C
- removed C18, C19, C20: 10pF, symbol Device:C
- removed C19, C20: 22uF, DIYSynthMNL:CP_Radial_D4.0mm_P1.50mm, symbol Device:C_Polarized
- removed C3, C4, C6, C7: 2.2uF, DIYSynthMNL:CP_Radial_D5.0mm_P2.50mm, symbol Device:C_Polarized
- removed D15, D16: ~, DIYSynthMNL:D_DO-41_SOD81_P7.62mm_Horizontal_BigPads, symbol Device:D
- removed D3, D4: 4148, symbol Device:D
- removed J10: SINE, DIYSynthMNL:AudioJack_3.5mm_long_pads, symbol DIYSynthMNL:PJ3001F
- removed J11: PULSE, DIYSynthMNL:AudioJack_3.5mm_long_pads, symbol DIYSynthMNL:PJ3001F
- removed J3: EuroPower_JST_3P, DIYSynthMNL:Eurorack_power_jst_3P, symbol DIYSynthMNL:JST_Eurorack_power_3P
- removed J3: FM, DIYSynthMNL:AudioJack_3.5mm_long_pads, symbol DIYSynthMNL:PJ3001F
- removed J4: EURO_PWR_16P, DIYSynthMNL:IDC-Header_2x08_P2.54mm_Vertical, symbol DIYSynthMNL:EURO_PWR_16_PIN
- removed J4: PWM, DIYSynthMNL:AudioJack_3.5mm_long_pads, symbol DIYSynthMNL:PJ3001F
- removed J5: Sync, DIYSynthMNL:AudioJack_3.5mm_long_pads, symbol DIYSynthMNL:PJ3001F
- removed J6: vOct1, DIYSynthMNL:AudioJack_3.5mm_long_pads, symbol DIYSynthMNL:PJ3001F
- removed J7: vOct2, DIYSynthMNL:AudioJack_3.5mm_long_pads, symbol DIYSynthMNL:PJ3001F
- removed J8: SAW, DIYSynthMNL:AudioJack_3.5mm_long_pads, symbol DIYSynthMNL:PJ3001F
- removed J9: TRI, DIYSynthMNL:AudioJack_3.5mm_long_pads, symbol DIYSynthMNL:PJ3001F
- removed JP1: Course_tune_gnd, symbol Jumper:Jumper_2_Open
- removed JP2: Course_tune_-5V, symbol Jumper:Jumper_2_Open
- removed R1, R2: *10K, DIYSynthMNL:R_quarter_watt_L6.3mm_D2.5mm_P7.62mm, symbol Device:R
- removed R10, R7: 470R, symbol Device:R
- removed R11, R12, R16, R19, R21, R22, R24, R28, R33, R34: 100K, symbol Device:R
- removed R13: 47K, symbol Device:R
- removed R14, R6: 1M5, symbol Device:R
- removed R15: 470K, symbol Device:R
- removed R17: 200K, symbol Device:R
- removed R18, R26, R27, R32, R40: 1K, symbol Device:R
- removed R20: 10M, symbol Device:R
- removed R23, R30, R36: 91K, symbol Device:R
- removed R25, R29, R35: 240K, symbol Device:R
- removed R3: 24K, symbol Device:R
- removed R31: 180K, symbol Device:R
- removed R37: 15K, symbol Device:R
- removed R38: 22K, symbol Device:R
- removed R39: 150K, symbol Device:R
- removed R4: 5K6, symbol Device:R
- removed R5: 1K8, symbol Device:R
- removed R8: 1M, symbol Device:R
- removed R9: 220K, symbol Device:R
- removed RV1, RV4: 10K, symbol Device:R_Potentiometer_Trim
- removed RV2, RV3, RV5, RV7: 100K, symbol Device:R_Potentiometer
- removed RV6: 2K, symbol Device:R_Potentiometer_Trim
- removed SW1: SW_SPDT, symbol Switch:SW_SPDT
- removed U1: AS3340, symbol DIYSynthMNL:A3340
- removed U1: 78M05, Package_TO_SOT_SMD:TO-252-2, symbol Regulator_Linear:LM78M05_TO252
- removed U2: TL074, symbol Amplifier_Operational:TL074
- added J12: Main, symbol Connector:Conn_01x20_Pin
- added J13: Ctrl, symbol Connector:Conn_01x20_Socket
Connections:
- new net 3340_Control_Board/CB_+12V: J13.19 (Pin_19)
- new net 3340_Control_Board/CB_+5V: J13.17 (Pin_17)
- new net 3340_Control_Board/CB_-12V: J13.20 (Pin_20)
- new net 3340_Control_Board/CB_-5V: J13.18 (Pin_18)
- new net 3340_Control_Board/CB_GND: J13.13 (Pin_13), J13.14 (Pin_14), J13.15 (Pin_15), J13.16 (Pin_16)
- new net 3340_Control_Board/Course_tune: J13.3 (Pin_3)
- new net 3340_Control_Board/Fine_tune: J13.4 (Pin_4)
- new net 3340_Control_Board/Hard_sync: J13.7 (Pin_7)
- new net 3340_Control_Board/Lin_FM: J13.5 (Pin_5)
- new net 3340_Control_Board/PWM: J13.6 (Pin_6)
- new net 3340_Control_Board/Pulse: J13.12 (Pin_12)
- new net 3340_Control_Board/Saw: J13.9 (Pin_9)
- new net 3340_Control_Board/Sine: J13.11 (Pin_11)
- new net 3340_Control_Board/Soft_sync: J13.8 (Pin_8)
- new net 3340_Control_Board/Tri: J13.10 (Pin_10)
- new net 3340_Control_Board/V/OCT_1: J13.1 (Pin_1)
- new net 3340_Control_Board/V/OCT_2: J13.2 (Pin_2)
- new net 3340_main_board/+12V: J12.19 (Pin_19)
- new net 3340_main_board/+5V: J12.17 (Pin_17)
- new net 3340_main_board/-12V: J12.20 (Pin_20)
- new net 3340_main_board/-5V: J12.18 (Pin_18)
- new net 3340_main_board/Course_tune: J12.3 (Pin_3)
- new net 3340_main_board/Fine_tune: J12.4 (Pin_4)
- new net 3340_main_board/GND: J12.13 (Pin_13), J12.14 (Pin_14), J12.15 (Pin_15), J12.16 (Pin_16)
- new net 3340_main_board/Hard_sync: J12.7 (Pin_7)
- new net 3340_main_board/Lin_FM: J12.5 (Pin_5)
- new net 3340_main_board/PWM: J12.6 (Pin_6)
- new net 3340_main_board/Pulse: J12.12 (Pin_12)
- new net 3340_main_board/Saw: J12.9 (Pin_9)
- new net 3340_main_board/Sine: J12.11 (Pin_11)
- new net 3340_main_board/Soft_sync: J12.8 (Pin_8)
- new net 3340_main_board/Tri: J12.10 (Pin_10)
- new net 3340_main_board/V/OCT_1: J12.1 (Pin_1)
- new net 3340_main_board/V/OCT_2: J12.2 (Pin_2)
- no-connect marks 14 -> 0
Other:
- added sheet 3340_Control_Board (3340_Control_Board.kicad_sch)
- added sheet 3340_main_board (3340_main_board.kicad_sch)
- note removed: "**0V to 10.7V"
- note removed: "**0V to 4V"
- note removed: "**0V to 8V"
- note removed: "**Electric Druid 3340 chip page on calculating the outputs: Saw = VCC * (2/3) Tri = VCC * (1/3) Pulse = VCC - 1.3V"
- note removed: "*Optional Load Resistor"
- note removed: "+/- 5V"
- note removed: "+/-5V Regulators"
- note removed: "-3.425V to 4.697V"
- note removed: "0V to 3.82V"
- note removed: "0V to 4V"
- note removed: "10.362V to 13.638V"
- note removed: "10Vpp"
- note removed: "19.891mV to 3.988V"
- note removed: "Course tune"
- note removed: "Course tune pot range jumpers"
- note removed: "Fine tune"
- note removed: "Frequency Control Summing Node"
- note removed: "Gain = 2.09"
- note removed: "High Frequency Tracking Trim"
- note removed: "Inputs"
- note removed: "Lin FM Input"
- note removed: "Linear FM Input Bias Network"
- note removed: "Op Amp Power"
- note removed: "Outputs"
- note removed: "PWM Amount"
- note removed: "PWM Hysteresis"
- note removed: "PWM Input"
- note removed: "Power"
- note removed: "Scale trim"
- note removed: "Sine Amplitude Trim"
- note removed: "Summing node bias network"
- note removed: "Switch up = Soft Sync Switch down = Hard Sync"
- note removed: "Sync Input"
- note removed: "Tri to Sin Waveshaper"
- note removed: "VCO Core"

Commit message: assigned through hole footprints
Parts:
- J12: footprint (none) -> Connector_PinHeader_2.54mm:PinHeader_1x20_P2.54mm_Vertical
- J13: footprint (none) -> Connector_PinSocket_2.54mm:PinSocket_1x20_P2.54mm_Vertical
Changed lines of the file:
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@@
       (effects (font (size 1.27 1.27)) (justify left))
     )
-    (property "Footprint" "" (at 142.875 95.885 0)
+    (property "Footprint" "Connector_PinSocket_2.54mm:PinSocket_1x20_P2.54mm_Vertical" (at 142.875 95.885 0)
       (effects (font (size 1.27 1.27)) hide)
     )
@@
       (effects (font (size 1.27 1.27)))
     )
-    (property "Footprint" "" (at 144.145 95.885 0)
+    (property "Footprint" "Connector_PinHeader_2.54mm:PinHeader_1x20_P2.54mm_Vertical" (at 144.145 95.885 0)
       (effects (font (size 1.27 1.27)) hide)
     )
