File: kicad/3340_Control_Board.kicad_sch (KiCad schematic)
At the start: 17 parts, among them J1 FM, J2 PWM, J3 Sync, J4 vOct1, J5 vOct2, J6 SAW, J7 TRI, J8 SINE, J9 PULSE, SW1 SW_SPDT

Commit message: assigned through hole footprints
Parts:
- C6: footprint (none) -> DIYSynthMNL:C_Rect_L7.0mm_W2.0mm_P5.00mm_BigPads
- JP3: footprint (none) -> Connector_PinHeader_2.54mm:PinHeader_1x03_P2.54mm_Vertical
- R7: footprint (none) -> DIYSynthMNL:R_quarter_watt_L6.3mm_D2.5mm_P7.62mm
- RV2, RV3, RV4, RV5: footprint (none) -> DIYSynthMNL:Potentiometer_RV09_BigPads
- SW1: footprint (none) -> DIYSynthMNL:ToggleSwitch_MTS-102_SPDT
Changed lines of the file:
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@@
       (effects (font (size 1.27 1.27)))
     )
-    (property "Footprint" "" (at 171.45 78.105 0)
+    (property "Footprint" "DIYSynthMNL:Potentiometer_RV09_BigPads" (at 171.45 78.105 0)
       (effects (font (size 1.27 1.27)) hide)
     )
@@
       (effects (font (size 1.27 1.27)))
     )
-    (property "Footprint" "" (at 81.915 116.713 90)
+    (property "Footprint" "DIYSynthMNL:R_quarter_watt_L6.3mm_D2.5mm_P7.62mm" (at 81.915 116.713 90)
       (effects (font (size 1.27 1.27)) hide)
     )
@@
       (effects (font (size 1.27 1.27)))
     )
-    (property "Footprint" "" (at 86.995 152.4 0)
+    (property "Footprint" "DIYSynthMNL:ToggleSwitch_MTS-102_SPDT" (at 86.995 152.4 0)
       (effects (font (size 1.27 1.27)) hide)
     )
@@
       (effects (font (size 1.27 1.27)) (justify right))
     )
-    (property "Footprint" "" (at 84.455 126.365 0)
+    (property "Footprint" "DIYSynthMNL:Potentiometer_RV09_BigPads" (at 84.455 126.365 0)
       (effects (font (size 1.27 1.27)) hide)
     )
@@
       (effects (font (size 1.27 1.27)) (justify right))
     )
-    (property "Footprint" "" (at 85.09 93.345 0)
+    (property "Footprint" "DIYSynthMNL:Potentiometer_RV09_BigPads" (at 85.09 93.345 0)
       (effects (font (size 1.27 1.27)) hide)
     )
@@
       (effects (font (size 1.27 1.27)))
     )
-    (property "Footprint" "" (at 81.915 151.4348 0)
+    (property "Footprint" "DIYSynthMNL:C_Rect_L7.0mm_W2.0mm_P5.00mm_BigPads" (at 81.915 151.4348 0)
       (effects (font (size 1.27 1.27)) hide)
     )
@@
       (effects (font (size 1.27 1.27)))
     )
-    (property "Footprint" "" (at 140.335 76.835 0)
+    (property "Footprint" "DIYSynthMNL:Potentiometer_RV09_BigPads" (at 140.335 76.835 0)
       (effects (font (size 1.27 1.27)) hide)
     )
@@
       (effects (font (size 1.27 1.27)))
     )
-    (property "Footprint" "" (at 140.335 85.725 0)
-      (effects (font (size 1.27 1.27)) hide)
-    )
+    (property "Footprint" "Connector_PinHeader_2.54mm:PinHeader_1x03_P2.54mm_Vertical" (at 140.335 85.725 0)
+      (effects (font (size 1.27 1.27)) hide)
+    )
