File: kicad/3340_main_board.kicad_sch (KiCad schematic)
At the start: 70 parts, among them U2 AS3340, U2 TL074

Commit message: assigned through hole footprints
Parts:
- C1, C2, C3, C4, C5, C7: footprint (none) -> DIYSynthMNL:C_Rect_L7.0mm_W2.0mm_P5.00mm_BigPads
- C10, C8, C9: footprint (none) -> Capacitor_THT:C_Disc_D3.0mm_W2.0mm_P2.50mm
- D1, D2: footprint (none) -> DIYSynthMNL:D_4148_BigPads
- R1, R10, R11, R12, R13, R14, R15, R16, R17, R18, R19, R2, R20, R21, R22, R23, R24, R25, R26, R27, R28, R29, R3, R30, R31, R32, R33, R34, R35, R36, R37, R38, R4, R5, R6, R8, R9: footprint (none) -> DIYSynthMNL:R_quarter_watt_L6.3mm_D2.5mm_P7.62mm
- RV1, RV6, RV7: footprint (none) -> DIYSynthMNL:Potentiometer_Bourns_3296W_Vertical_BigPads
- U2: footprint (none) -> DIYSynthMNL:DIP-14_W7.62mm_LongPads
- U2: footprint (none) -> Package_DIP:DIP-16_W7.62mm_Socket_LongPads
